File: pcb/PhoniESP32/I2S.kicad_sch (KiCad schematic)
At the start: 0 parts

Commit message: chore(pcb): wip
Parts:
- added U2: MAX98357AETE+T, JLCPCB:TQFN-16_L3.0-W3.0-P0.50-BL-EP1.5, symbol JLCPCB:MAX98357AETE+T
Changed lines of the file:
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@@
 	(generator_version "9.0")
 	(paper "A4")
+	(symbol
+		(lib_id "JLCPCB:MAX98357AETE+T")
+		(at 90.17 83.82 0)
+		(unit 1)
+		(exclude_from_sim no)
+		(in_bom yes)
+		(on_board yes)
+		(dnp no)
+		(fields_autoplaced yes)
+		(property "Reference" "U2"
+			(at 90.17 67.31 0)
+			(effects
+				(font
+					(size 1.27 1.27)
+				)
+			)
+		)
+		(property "Value" "MAX98357AETE+T"
+			(at 90.17 69.85 0)
+			(effects
+				(font
+					(size 1.27 1.27)
+				)
+			)
+		)
+		(property "Footprint" "JLCPCB:TQFN-16_L3.0-W3.0-P0.50-BL-EP1.5"
+			(at 90.17 105.41 0)
+			(effects
+				(font
+					(size 1.27 1.27)
+				)
+				(hide yes)
+			)
+		)
+		(property "Datasheet" ""
+			(at 90.17 83.82 0)
+			(effects
+				(font
+					(size 1.27 1.27)
+				)
+				(hide yes)
+			)
+		)
+		(property "Description" ""
+			(at 90.17 83.82 0)
+			(effects
+				(font
+					(size 1.27 1.27)
+				)
+				(hide yes)
+			)
+		)
+		(property "LCSC Part" "C910544"
+			(at 90.17 107.95 0)
+			(effects
+				(font
+					(size 1.27 1.27)
+				)
+				(hide yes)
+			)
+		)
+		(pin "13"
+		)
+		(pin "15"
+		)
+		(pin "8"
+		)
+		(pin "12"
+		)
+		(pin "9"
+		)
+		(pin "14"
+		)
+		(pin "11"
+		)
+		(pin "17"
+		)
+		(pin "5"
+		)
+		(pin "7"
+		)
+		(pin "10"
+		)
+		(pin "16"
+		)
+		(pin "4"
+		)
+		(pin "3"
+		)
+		(pin "2"
+		)
+		(pin "1"
+		)
+		(pin "6"
+		)
+		(instances
+			(project ""
+				(path "/a246d5c1-33d2-4ce4-8f5f-6a6b3acd3d9a/596f5b6c-eb79-41a3-bcdd-6fb80ece9deb"
+					(reference "U2")
+					(unit 1)
+				)
+			)
+		)
+	)
 )
