File: pcb/PhoniESP32/PhoniESP32.kicad_pcb (KiCad board)
At the start: 2 copper layers, 1 part, among them U1 ESP32-C6-MINI-1

Commit message: chore(pcb): wip
Parts:
- added D1: USBLC6-2SC6, JLCPCB:SOT-23-6_L2.9-W1.6-P0.95-LS2.8-BL, F.Cu at (118.1, 93.8)
- added J1: Connector, USB-TYPE-C-16P, PCM_JLCPCB:TYPE-C-SMD_HX-TYPE-C-16PIN, F.Cu at (110.1, 95.3)
- added J2: Conn_01x02_Pin, Connector_Wire:SolderWire-0.5sqmm_1x02_P4.8mm_D0.9mm_OD2.3mm, F.Cu at (107.1, 103.2)
- added R1: 5.1kΩ, PCM_JLCPCB:R_0603, F.Cu at (117.4, 97.1)
- added R2: 5.1kΩ, PCM_JLCPCB:R_0603, F.Cu at (117.4, 99.3)
- added TF1: TF-CARD H1.8, JLCPCB:TF-SMD_TF-CARD-H1.8, F.Cu at (113.5, 79.3)
- added U2: MAX98357AETE+T, JLCPCB:TQFN-16_L3.0-W3.0-P0.50-BL-EP1.5, F.Cu at (87.7, 97.9)
- added U3: ESP32-C6-MINI-1-N4, JLCPCB:WIFIM-SMD_61P-L16.6-W13.2-P0.80-ESP32-C6-MINI-1-N4, F.Cu at (94.0, 85.9)
- added U4: BQ24075RGTR, JLCPCB:QFN-16_L3.0-W3.0-P0.50-TL-EP1.7, F.Cu at (117.0, 103.5)
- U1: value ESP32-C6-MINI-1 -> TPS631000DRLR; footprint RF_Module:ESP32-C6-MINI-1 -> JLCPCB:SOT-583-8_L2.1-W1.2-P0.50-LS1.6-BL
- moved U1 81.6 mm to (106.5, 106.9)
Connections:
- U1 pad 1: Net-(U1-GND-Pad1) -> unconnected-(U1-VOUT-Pad1)
- U1 pad 2: Net-(U1-GND-Pad1) -> unconnected-(U1-LX2-Pad2)
