File: pcb/PhoniESP32/PhoniESP32.kicad_sch (KiCad schematic)
At the start: 1 part, among them U1 ESP32-C6-MINI-1

Commit message: chore(pcb): wip
Parts:
- removed U1: ESP32-C6-MINI-1, RF_Module:ESP32-C6-MINI-1, symbol RF_Module:ESP32-C6-MINI-1
- added U3: ESP32-C6-MINI-1-N4, JLCPCB:WIFIM-SMD_61P-L16.6-W13.2-P0.80-ESP32-C6-MINI-1-N4, symbol JLCPCB:ESP32-C6-MINI-1-N4
Changed lines of the file:
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@@
 	(paper "A4")
 	(symbol
-		(lib_id "RF_Module:ESP32-C6-MINI-1")
-		(at 146.05 83.82 0)
+		(lib_id "JLCPCB:ESP32-C6-MINI-1-N4")
+		(at 213.36 83.82 0)
 		(unit 1)
 		(exclude_from_sim no)
@@
 		(dnp no)
 		(fields_autoplaced yes)
-		(property "Reference" "U1"
-			(at 148.1933 55.88 0)
+		(property "Reference" "U3"
+			(at 213.36 43.18 0)
 			(effects
 				(font
 					(size 1.27 1.27)
 				)
-				(justify left)
 			)
 		)
-		(property "Value" "ESP32-C6-MINI-1"
-			(at 148.1933 58.42 0)
+		(property "Value" "ESP32-C6-MINI-1-N4"
+			(at 213.36 45.72 0)
 			(effects
 				(font
 					(size 1.27 1.27)
 				)
-				(justify left)
 			)
 		)
-		(property "Footprint" "RF_Module:ESP32-C6-MINI-1"
-			(at 163.83 109.22 0)
+		(property "Footprint" "JLCPCB:WIFIM-SMD_61P-L16.6-W13.2-P0.80-ESP32-C6-MINI-1-N4"
+			(at 213.36 124.46 0)
 			(effects
 				(font
@@
 			)
 		)
-		(property "Datasheet" "https://www.espressif.com/sites/default/files/documentation/esp32-c6-mini-1_mini-1u_datasheet_en.pdf"
-			(at 146.05 46.99 0)
+		(property "Datasheet" ""
+			(at 213.36 83.82 0)
 			(effects
 				(font
@@
 			)
 		)
-		(property "Description" "RF Module, ESP32-C6 SoC, Wi-Fi 802.11b/g/n/ax, Bluetooth, BLE, Zigbee, Thread, 32-bit, 3.3V, SMD, onboard antenna"
-			(at 146.05 44.45 0)
+		(property "Description" ""
+			(at 213.36 83.82 0)
 			(effects
 				(font
@@
 			)
 		)
-		(pin "53"
+		(property "LCSC Part" "C5736265"
+			(at 213.36 127 0)
+			(effects
+				(font
+					(size 1.27 1.27)
+				)
+				(hide yes)
+			)
+		)
+		(pin "29"
+		)
+		(pin "15"
+		)
+		(pin "35"
+		)
+		(pin "51"
+		)
+		(pin "44"
+		)
+		(pin "18"
 		)
 		(pin "42"
 		)
-		(pin "40"
+		(pin "39"
 		)
-		(pin "29"
+		(pin "12"
 		)
-		(pin "7"
+		(pin "37"
 		)
-		(pin "48"
-		)
-		(pin "33"
-		)
-		(pin "43"
+		(pin "28"
 		)
 		(pin "9"
 		)
+		(pin "14"
+		)
+		(pin "16"
+		)
+		(pin "31"
+		)
+		(pin "30"
+		)
 		(pin "46"
+		)
+		(pin "50"
+		)
+		(pin "47"
+		)
+		(pin "34"
+		)
+		(pin "49"
+		)
+		(pin "10"
+		)
+		(pin "40"
+		)
+		(pin "20"
+		)
+		(pin "19"
+		)
+		(pin "21"
 		)
 		(pin "26"
 		)
-		(pin "51"
-		)
-		(pin "1"
-		)
-		(pin "52"
-		)
-		(pin "47"
-		)
-		(pin "49"
-		)
-		(pin "50"
+		(pin "36"
 		)
 		(pin "38"
 		)
-		(pin "21"
-		)
-		(pin "45"
-		)
-		(pin "18"
-		)
-		(pin "19"
-		)
-		(pin "28"
-		)
-		(pin "16"
-		)
-		(pin "10"
-		)
 		(pin "13"
 		)
-		(pin "32"
-		)
-		(pin "15"
-		)
-		(pin "44"
-		)
-		(pin "39"
-		)
-		(pin "24"
-		)
-		(pin "6"
-		)
-		(pin "27"
-		)
-		(pin "5"
-		)
-		(pin "30"
-		)
-		(pin "11"
-		)
-		(pin "37"
-		)
-		(pin "31"
-		)
-		(pin "35"
+		(pin "17"
 		)
 		(pin "25"
+		)
+		(pin "53"
 		)
 		(pin "4"
@@
 		(pin "3"
 		)
-		(pin "23"
+		(pin "2"
 		)
-		(pin "34"
+		(pin "1"
 		)
-		(pin "17"
+		(pin "8"
+		)
+		(pin "24"
+		)
+		(pin "7"
+		)
+		(pin "41"
+		)
+		(pin "6"
+		)
+		(pin "5"
+		)
+		(pin "33"
 		)
 		(pin "22"
 		)
-		(pin "36"
+		(pin "32"
 		)
-		(pin "14"
+		(pin "27"
 		)
-		(pin "2"
+		(pin "11"
 		)
-		(pin "12"
+		(pin "48"
 		)
-		(pin "8"
+		(pin "43"
 		)
-		(pin "20"
+		(pin "23"
 		)
-		(pin "41"
+		(pin "52"
+		)
+		(pin "45"
 		)
 		(instances
 			(project ""
 				(path "/a246d5c1-33d2-4ce4-8f5f-6a6b3acd3d9a"
-					(reference "U1")
+					(reference "U3")
 					(unit 1)
 				)

Commit message: chore(pcb): power, mcu, spi wip
Parts:
- added C6: 22uF, PCM_JLCPCB:C_0603, symbol PCM_JLCPCB-Capacitors:0603,22uF
- added C7: 100nF, PCM_JLCPCB:C_0402, symbol PCM_JLCPCB-Capacitors:0402,100nF
- added D4: Green, PCM_JLCPCB:D_0805, symbol PCM_JLCPCB-Diodes:LED,0805,Green
- added J3: Conn_Buttons, Connector_PinHeader_2.54mm:PinHeader_1x05_P2.54mm_Vertical, symbol Connector:Conn_01x05_Pin
- added R13: 150Ω, PCM_JLCPCB:R_0603, symbol PCM_JLCPCB-Resistors:0603,150Ω
- added S1, S2: Tactile Button, 160gf, PCM_JLCPCB:SW_TS-1088-AR02016, symbol PCM_JLCPCB-Connectors_Buttons:Tactile Button, 160gf, 12V, 50mA, 4.0mm
Connections:
- net GND: now reaches U3.1 (GND)
- net GND: now also U3.11 (GND), U3.14 (GND), U3.2 (GND), U3.36 (GND), U3.37 (GND), U3.38 (GND), U3.39 (GND), U3.40 (GND), U3.41 (GND), U3.42 (GND), U3.43 (GND), U3.44 (GND), U3.45 (GND), U3.46 (GND), U3.47 (GND), U3.48 (GND), U3.49 (GND), U3.50 (GND), U3.51 (GND), U3.52 (GND), U3.53 (GND), C6.2, C7.2, D4.1, J3.1 (Pin_1), S1.1 (A), S2.1 (A)
- net BTN_PLAY: now reaches U3.12 (IO0)
- net BTN_PLAY: now also J3.2 (Pin_2)
- net BTN_NEXT: now reaches U3.13 (IO1)
- net BTN_NEXT: now also J3.3 (Pin_3)
- net USB_D-: now reaches U3.17 (IO12)
- net USB_D+: now reaches U3.18 (IO13)
- net at U3.22 (IO8): now also R13.1
- net ESP_BOOT: now reaches U3.23 (IO9)
- net ESP_BOOT: now also S2.2 (B)
- net +3.3V: now reaches U3.3 (3V3)
- net +3.3V: now also C6.1, C7.1
- net BTN_VOL_DOWN: now reaches U3.5 (IO2)
- net BTN_VOL_DOWN: now also J3.4 (Pin_4)
- net BTN_VOL_UP: now reaches U3.6 (IO3)
- net BTN_VOL_UP: now also J3.5 (Pin_5)
- net ESP_EN: now reaches U3.8 (EN)
- net ESP_EN: now also S1.2 (B)
- new net: D4.2, R13.2
- no-connect marks 0 -> 9
Other:
- sheet Power ports: added CHG, USB_DN, USB_DP; removed none
