File: pcb/PhoniESP32/Power.kicad_sch (KiCad schematic)
At the start: 0 parts

Commit message: chore(pcb): wip
Parts:
- added D1: USBLC6-2SC6, JLCPCB:SOT-23-6_L2.9-W1.6-P0.95-LS2.8-BL, symbol JLCPCB:USBLC6-2SC6
- added J1: Connector, USB-TYPE-C-16P, PCM_JLCPCB:TYPE-C-SMD_HX-TYPE-C-16PIN, symbol PCM_JLCPCB-Extended:Connector, USB-TYPE-C-16P
- added J2: Conn_01x02_Pin, Connector_Wire:SolderWire-0.5sqmm_1x02_P4.8mm_D0.9mm_OD2.3mm, symbol Connector:Conn_01x02_Pin
- added R1, R2: 5.1kΩ, PCM_JLCPCB:R_0603, symbol PCM_JLCPCB-Resistors:0603,5.1kΩ
- added U1: TPS631000DRLR, JLCPCB:SOT-583-8_L2.1-W1.2-P0.50-LS1.6-BL, symbol JLCPCB:TPS631000DRLR
- added U4: BQ24075RGTR, JLCPCB:QFN-16_L3.0-W3.0-P0.50-TL-EP1.7, symbol JLCPCB:BQ24075RGTR
Connections:
- new net: J1.A5 (CC1), R1.1
- new net: D1.1, J1.A7 (D-), J1.B7 (D-)
- new net: D1.3, J1.A6 (D+), J1.B6 (D+)
- new net: J2.1 (Pin_1), U4.2 (BAT)
- new net: J2.2 (Pin_2), U4.3 (BAT)
- new net: J1.B5 (CC2), R2.1
- new net GND: D1.2, J1.A12B1 (GND), J1.B12A1 (GND), J1.S1 (SHIELD), R1.2, R2.2
- new net USB_DN: D1.6
- new net USB_DP: D1.4
- new net VBUS: D1.5, J1.A9B4 (VBUS), J1.B9A4 (VBUS)
- no-connect marks 0 -> 2

Commit message: chore(pcb): power, mcu, spi wip
Parts:
- added C1: 1uF, PCM_JLCPCB:C_0603, symbol PCM_JLCPCB-Capacitors:0603,1uF
- added C2, C3: 10uF, PCM_JLCPCB:C_0603, symbol PCM_JLCPCB-Capacitors:0603,10uF
- added C4: 22uF, PCM_JLCPCB:C_0603, symbol PCM_JLCPCB-Capacitors:0603,22uF
- added C5: 47uF, PCM_JLCPCB:C_0805, symbol PCM_JLCPCB-Capacitors:0805,47uF
- added D2: Red, PCM_JLCPCB:D_0603, symbol PCM_JLCPCB-Diodes:LED,0603,Red
- added D3: Yellow, PCM_JLCPCB:D_0603, symbol PCM_JLCPCB-Diodes:LED,0603,Yellow
- added L1: DFE252012P-1R0M=P2, JLCPCB:L1008, symbol JLCPCB:DFE252012P-1R0M=P2
- added R10, R11, R6, R7: 1kΩ, PCM_JLCPCB:R_0603, symbol PCM_JLCPCB-Resistors:0603,1kΩ
- added R12, R4, R5: 1.5kΩ, PCM_JLCPCB:R_0603, symbol PCM_JLCPCB-Resistors:0603,1.5kΩ
- added R3: 10kΩ, PCM_JLCPCB:R_0603, symbol PCM_JLCPCB-Resistors:0603,10kΩ
- added R8: 91kΩ, PCM_JLCPCB:R_0603, symbol PCM_JLCPCB-Resistors:0603,91kΩ
- added R9: 510kΩ, PCM_JLCPCB:R_0603, symbol PCM_JLCPCB-Resistors:0603,510kΩ
- J2: value Conn_01x02_Pin -> Conn_Battery; footprint Connector_Wire:SolderWire-0.5sqmm_1x02_P4.8mm_D0.9mm_OD2.3mm -> Connector_PinHeader_2.54mm:PinHeader_1x02_P2.54mm_Vertical; now not fitted; now left out of the parts list
Connections:
- net GND: now also J2.2 (Pin_2), U1.6 (MODE), U1.7 (GND), U4.15 (SYSOFF), U4.17 (EP), U4.4 (#CE), U4.6 (EN1), U4.8 (VSS), C1.2, C2.1, C3.2, C4.2, C5.2, R11.2, R12.1, R3.1, R5.1, R8.2
- net VBUS: now also U4.13 (IN), C1.1, R10.1
- net at J2.1 (Pin_1), U4.2 (BAT): now also U4.3 (BAT), C2.2
- net +3.3V: now reaches U1.1 (VOUT)
- net +3.3V: now also C5.1, R9.1
- net at U1.2 (LX2): now also L1.2
- net at U1.3 (LX1): now also L1.1
- net +5V: now reaches U1.4 (VIN)
- net +5V: now also U1.5 (EN), U4.10 (OUT), U4.11 (OUT), U4.5 (EN2), C3.1, C4.1, R6.2, R7.2
- net at U1.8 (FB): now also R8.1, R9.2
- net at U4.1 (TS): now also R3.2
- net at U4.12 (ILIM): now also R5.2
- net at U4.16 (ISET): now also R4.2
- net at U4.7 (#PGOOD): now also D2.1
- net at U4.9 (#CHG): now also D3.1
- new net: D2.2, R6.1
- new net: D3.2, R7.1
- new net: R12.2, R4.1
- new net CHG: R10.2, R11.1
- no-connect marks 2 -> 3
Other:
- moved on the sheet: U1, U4
