File: pcb/PhoniESP32/Power.kicad_sch (KiCad schematic)
At the start: 30 parts, among them J1 Connector, USB-TYPE-C-16P, J2 Conn_Battery, SW1 SK12D07VG5, U1 TPS631000DRLR, U5 BQ24073RGTR

Commit message: feat(pcb): version for hand soldering
Parts:
- removed R8: 91kΩ, PCM_JLCPCB:R_0603, symbol PCM_JLCPCB-Resistors:0603,91kΩ
- removed R9: 510kΩ, PCM_JLCPCB:R_0603, symbol PCM_JLCPCB-Resistors:0603,510kΩ
- added R8: 510kΩ, PCM_JLCPCB:R_0603, symbol PCM_JLCPCB-Resistors:0603,510kΩ
- added R9: 91kΩ, PCM_JLCPCB:R_0603, symbol PCM_JLCPCB-Resistors:0603,91kΩ
- C1: Notes 1-10 uF -> (none)
- D1: MPN (none) -> USBLC6-2SC6
- D2: footprint PCM_JLCPCB:D_0603 -> PCM_JLCPCB:D_0805; symbol PCM_JLCPCB-Diodes:LED,0603,Red -> PCM_JLCPCB-Diodes:LED,0805,Red; Category Optocouplers & LEDs & Infrared,Light Emitting Diodes (LED) -> Optoelectronics,Light Emitting Diodes (LED); Diode Configuration (none) -> Independent Diode; Dominant Wavelength (none) -> 615nm~630nm; Emitted Color (none) -> Red; Forward Current (none) -> 25mA; Forward Voltage (VF) (none) -> 1.6V~2.6V; LCSC C2286 -> C84256; Lens Color (none) -> Colorless Transparent Lens; Luminous Intensity (none) -> 67mcd~195mcd; MPN (none) -> NCD0805R1; Manufacturer Hubei KENTO Elec -> Foshan NationStar Optoelectronics; Operating Temperature (none) -> -30°C~+85°C; Part KT-0603R -> NCD0805R1; Power Dissipation (none) -> 65mW; Price 0.009USD -> 0.016USD; Stock 5373336 -> 2976925; Viewing Angle (none) -> 130°
- D3: footprint PCM_JLCPCB:D_0603 -> PCM_JLCPCB:D_0805; symbol PCM_JLCPCB-Diodes:LED,0603,Yellow -> PCM_JLCPCB-Diodes:LED,0805,Yellow; Attrition Qty 6 -> 10; Category Optoelectronics,Light Emitting Diodes (LED) -> Optocouplers & LEDs & Infrared,Light Emitting Diodes (LED); Class Preferred Component -> Basic Component; LCSC C89811 -> C2296; MPN (none) -> KT-0805Y; Manufacturer Foshan NationStar Optoelectronics -> Hubei KENTO Elec; Part NCD0603Y2 -> KT-0805Y; Price 0.021USD -> 0.015USD; Stock 109176 -> 662678
- J1: MPN (none) -> USB-TYPE-C-019
- J2: footprint Connector_PinHeader_2.54mm:PinHeader_1x02_P2.54mm_Vertical -> Connector_JST:JST_PH_B2B-PH-K_1x02_P2.00mm_Vertical; LCSC Part (none) -> C131337; MPN (none) -> B2B-PH-K-S(LF)(SN)
- L1: MPN (none) -> DFE252012P-1R0M=P2
- SW1: MPN (none) -> SK12D07VG5
- U1: MPN (none) -> TPS631000DRLR
- U5: MPN (none) -> BQ24073RGTR
Connections:
- net +3.3V: now also R8.1
- net GND: now also C2.2, J2.1 (Pin_1), R9.2; no longer C2.1, J2.2 (Pin_2)
- net at U1.8 (FB): now also R8.2, R9.1
- net BAT+: now reaches U5.2 (BAT), U5.3 (BAT)
- net BAT+: now also C2.1, J2.2 (Pin_2); no longer C2.2, J2.1 (Pin_1)
- net VIN: now reaches C3.1, SW1.2, TP5.1, U5.10 (OUT), U5.11 (OUT), U5.5 (EN2)
- net VIN: now also R6.1, R7.1
- net +5V renamed VIN_SW
- net VIN_SW: no longer R6.1, R7.1
Other:
- title: (none) -> PhoniESP32
- moved on the sheet: C2, C4, J2, TP5
