File: pcb/PhoniESP32/SPI.kicad_sch (KiCad schematic)
At the start: 0 parts

Commit message: chore(pcb): wip
Parts:
- added TF1: TF-CARD H1.8, JLCPCB:TF-SMD_TF-CARD-H1.8, symbol JLCPCB:TF-CARDH1.8
Changed lines of the file:
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@@
 	(generator_version "9.0")
 	(paper "A4")
+	(symbol
+		(lib_id "JLCPCB:TF-CARDH1.8")
+		(at 54.61 66.04 0)
+		(unit 1)
+		(exclude_from_sim no)
+		(in_bom yes)
+		(on_board yes)
+		(dnp no)
+		(fields_autoplaced yes)
+		(property "Reference" "TF1"
+			(at 53.34 45.72 0)
+			(effects
+				(font
+					(size 1.27 1.27)
+				)
+			)
+		)
+		(property "Value" "TF-CARD H1.8"
+			(at 53.34 48.26 0)
+			(effects
+				(font
+					(size 1.27 1.27)
+				)
+			)
+		)
+		(property "Footprint" "JLCPCB:TF-SMD_TF-CARD-H1.8"
+			(at 54.61 81.28 0)
+			(effects
+				(font
+					(size 1.27 1.27)
+				)
+				(hide yes)
+			)
+		)
+		(property "Datasheet" ""
+			(at 54.61 66.04 0)
+			(effects
+				(font
+					(size 1.27 1.27)
+				)
+				(hide yes)
+			)
+		)
+		(property "Description" ""
+			(at 54.61 66.04 0)
+			(effects
+				(font
+					(size 1.27 1.27)
+				)
+				(hide yes)
+			)
+		)
+		(property "LCSC Part" "C7529389"
+			(at 54.61 83.82 0)
+			(effects
+				(font
+					(size 1.27 1.27)
+				)
+				(hide yes)
+			)
+		)
+		(pin "12"
+		)
+		(pin "13"
+		)
+		(pin "1"
+		)
+		(pin "2"
+		)
+		(pin "5"
+		)
+		(pin "7"
+		)
+		(pin "3"
+		)
+		(pin "8"
+		)
+		(pin "10"
+		)
+		(pin "9"
+		)
+		(pin "11"
+		)
+		(pin "6"
+		)
+		(pin "4"
+		)
+		(instances
+			(project ""
+				(path "/a246d5c1-33d2-4ce4-8f5f-6a6b3acd3d9a/fe612abb-b371-4c9e-9c6b-73258b810d1f"
+					(reference "TF1")
+					(unit 1)
+				)
+			)
+		)
+	)
 )

Commit message: chore(pcb): power, mcu, spi wip
Parts:
- added C8: 22uF, PCM_JLCPCB:C_0603, symbol PCM_JLCPCB-Capacitors:0603,22uF
- added C9: 100nF, PCM_JLCPCB:C_0402, symbol PCM_JLCPCB-Capacitors:0402,100nF
- added J4: Conn_MFRC522, Connector_PinSocket_2.54mm:PinSocket_1x06_P2.54mm_Vertical, symbol Connector:Conn_01x06_Pin
- added R14, R15: 10kΩ, PCM_JLCPCB:R_0603, symbol PCM_JLCPCB-Resistors:0603,10kΩ
Connections:
- net at TF1.1 (DAT2): now also R15.1
- net GND: now reaches TF1.10 (GND)
- net GND: now also TF1.11 (GND), TF1.12 (GND), TF1.13 (GND), TF1.6 (VSS), C8.2, C9.2
- net SD_CS: now reaches TF1.2 (CD/DAT3)
- net MOSI: now reaches TF1.3 (CMD)
- net +3.3V: now reaches TF1.4 (VDD)
- net +3.3V: now also C8.1, C9.1, R14.2, R15.2
- net SCLK: now reaches TF1.5 (CLK)
- net MISO: now reaches TF1.7 (DAT0)
- net at TF1.8 (DAT1): now also R14.1
- no-connect marks 0 -> 1
Other:
- moved on the sheet: TF1
